File: device/*/*.kicad_pcb (KiCad board)
At the start: 2 copper layers, 99.5 x 99.5 mm, 7 parts, among them SW1 SW_Push, SW2 SW_Push

Commit message: pcb
Connections:
- DS2 pad 1: Net-(DS2-LED(+)) -> Net-(DS2-LED(-))
- DS2 pad 2: Net-(DS2-LED(-)) -> Net-(DS2-LED(+))
- DS2 pad 5: Net-(DS2-LED(+)) -> Net-(DS2-LED(-))
- Esp32-Wroom-32D1 pad 2: Net-(DS2-LED(-)) -> Net-(DS2-LED(+))
- Esp32-Wroom-32D1 pad 38: Net-(DS2-LED(+)) -> Net-(DS2-LED(-))
- R3 pad 1: Net-(DS2-LED(+)) -> Net-(DS2-LED(-))
Routing:
- net Net-(DS2-LED(+)): track 67.4 -> 53.2 mm
- net Net-(DS2-LED(-)): track 56.6 -> 69.9 mm
- net Net-(DS2-RS): track 18.4 -> 19.1 mm
