File: device/*/*.kicad_sch (KiCad schematic)
At the start: 1 part, among them U1 ESP32-WROOM-32D

Commit message: pcb
Parts:
- removed U1: ESP32-WROOM-32D, RF_Module:ESP32-WROOM-32D, symbol RF_Module:ESP32-WROOM-32D
- added D1: LED, LED_THT:LED_D5.0mm, symbol Device:LED
- added DS2: WC1602A, Display:WC1602A, symbol Display_Character:WC1602A
- added Esp32-Wroom-32D1: ~, esp32_footprint:esp32_my_footpring, symbol my_stuff:esp32-wroom-32d_my_version
- added R2, R3: R, Resistor_THT:R_Axial_DIN0207_L6.3mm_D2.5mm_P7.62mm_Horizontal, symbol Device:R
- added SW1, SW2: SW_Push, Button_Switch_THT:SW_PUSH_6mm_H5mm, symbol Switch:SW_Push
Connections:
- new net: D1.1 (K), R2.1
- new net: D1.2 (A), Esp32-Wroom-32D1.12 (D27)
- new net: Esp32-Wroom-32D1.1 (GND), R2.2, SW1.2, SW2.2
- new net: Esp32-Wroom-32D1.13 (D14), SW1.1
- new net: DS2.16 (LED(-)), DS2.2 (VDD), Esp32-Wroom-32D1.2 (3V3)
- new net: DS2.4 (RS), Esp32-Wroom-32D1.23 (D15)
- new net: DS2.6 (E), Esp32-Wroom-32D1.24 (D2)
- new net: DS2.11 (D4), Esp32-Wroom-32D1.26 (D4)
- new net: DS2.12 (D5), Esp32-Wroom-32D1.27 (D16)
- new net: DS2.13 (D6), Esp32-Wroom-32D1.28 (D17)
- new net: DS2.14 (D7), Esp32-Wroom-32D1.29 (D5)
- new net: DS2.1 (VSS), DS2.15 (LED(+)), DS2.5 (R/W), Esp32-Wroom-32D1.38 (GND), R3.1
- new net: Esp32-Wroom-32D1.8 (D32), SW2.1
- new net: DS2.3 (VO), R3.2
- no-connect marks 0 -> 22

Commit message: pcb
Connections:
- net at DS2.2 (VDD), Esp32-Wroom-32D1.2 (3V3): now also DS2.15 (LED(+)); no longer DS2.16 (LED(-))
- net at DS2.1 (VSS), DS2.5 (R/W), Esp32-Wroom-32D1.38 (GND)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: now also DS2.16 (LED(-)); no longer DS2.15 (LED(+))
Changed lines of the file:
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@@
 	(paper "A4")
 	(junction
+		(at 127 76.2)
+		(diameter 0)
+		(color 0 0 0 0)
+	)
+	(junction
 		(at 116.84 76.2)
 		(diameter 0)
@@
 	)
 	(junction
-		(at 129.54 76.2)
+		(at 129.54 78.74)
 		(diameter 0)
 		(color 0 0 0 0)
@@
 		(color 0 0 0 0)
 	)
-	(junction
-		(at 127 78.74)
-		(diameter 0)
-		(color 0 0 0 0)
-	)
 	(no_connect
 		(at 34.29 45.72)
@@
 	(wire
 		(pts
-			(xy 68.58 78.74) (xy 127 78.74)
-		)
-		(stroke
-			(width 0)
-			(type default)
-		)
-	)
-	(wire
-		(pts
-			(xy 132.08 76.2) (xy 129.54 76.2)
-		)
-		(stroke
-			(width 0)
-			(type default)
-		)
-	)
-	(wire
-		(pts
 			(xy 96.52 33.02) (xy 96.52 76.2)
 		)
@@
 	(wire
 		(pts
-			(xy 129.54 38.1) (xy 129.54 76.2)
-		)
-		(stroke
-			(width 0)
-			(type default)
-		)
-	)
-	(wire
-		(pts
 			(xy 34.29 66.04) (xy 33.02 66.04)
 		)
@@
 	(wire
 		(pts
-			(xy 127 40.64) (xy 127 78.74)
+			(xy 127 76.2) (xy 132.08 76.2)
 		)
 		(stroke
@@
 	(wire
 		(pts
+			(xy 129.54 38.1) (xy 129.54 78.74)
+		)
+		(stroke
+			(width 0)
+			(type default)
+		)
+	)
+	(wire
+		(pts
+			(xy 129.54 78.74) (xy 134.62 78.74)
+		)
+		(stroke
+			(width 0)
+			(type default)
+		)
+	)
+	(wire
+		(pts
 			(xy 33.02 66.04) (xy 33.02 38.1)
 		)
@@
 	(wire
 		(pts
-			(xy 116.84 76.2) (xy 129.54 76.2)
+			(xy 116.84 76.2) (xy 127 76.2)
 		)
 		(stroke
@@
 	(wire
 		(pts
-			(xy 134.62 78.74) (xy 127 78.74)
-		)
-		(stroke
+			(xy 127 40.64) (xy 127 76.2)
+		)
+		(stroke
+			(width 0)
+			(type default)
+		)
+	)
+	(wire
+		(pts
+			(xy 68.58 78.74) (xy 129.54 78.74)
+		)
+		(stroke
